File: adapter/circuit/circuit.brd (EAGLE design)
At the start: 33 x 38 mm, 11 parts, among them IC1 TS 5205 CX533, Q1 BSS123

Commit message: update to V1.5
Parts:
- JP1: device pinhead:1X05 -> pinhead:1X04
- R3: value 10K -> 5K
- moved JP1 1.27 mm to (16.5, 10.8), flipped to the top
Connections:
- net RX_5V: now also JP1.4; no longer JP1.1
- net TX_5V: now also JP1.1; no longer JP1.5
Routing:
- net GND: track 34.2 -> 42.3 mm
- net +5V: track 22.5 -> 27.0 mm
- net RX_5V: track 21.7 -> 23.5 mm
- net TX_5V: track 3.34 -> 5.15 mm
- net N$9: track 3.70 -> 5.23 mm
- net N$10: track 3.70 -> 5.23 mm
Other:
- board text added: "V1.5"
- board text removed: "V1.4"
