File: adapter/circuit/circuit.sch (EAGLE design)
At the start: 11 parts, among them IC1 TS 5205 CX533, Q1 BSS123

Commit message: update to V1.5
Parts:
- JP1: device pinhead:PINHD-1X5 -> pinhead:PINHD-1X4
- R3: value 10K -> 5K
Connections:
- net RX_5V: now also JP1.4; no longer JP1.1
- net TX_5V: now also JP1.1; no longer JP1.5
Other:
- note added: "V 1.5"
- note removed: "NC"
- note removed: "V 1.4"
